File: adapter-shield/adapter-shield.sch (KiCad schematic (older format))
At the start: 74 parts, among them J1 Camera, U1 AP1117-33

Commit message: Part nums and footprints
Parts:
- removed Q?: Q_NMOS_GSD, symbol Device:Q_NMOS_GSD
- added Q10: Q_PMOS_GSD, Package_TO_SOT_SMD:SOT-23, symbol Device:Q_PMOS_GSD
- BT1: renamed from BT?; footprint (none) -> Connector_AMASS:AMASS_XT60-M_1x02_P7.20mm_Vertical
- C1: renamed from C3; footprint (none) -> Capacitor_THT:C_Radial_D6.3mm_H7.0mm_P2.50mm; Digikey Part Num (none) -> 1189-2182-ND
- C2, C3: renamed from C?; footprint (none) -> Capacitor_SMD:CP_Elec_8x5.4; Digikey Part Num (none) -> 493-2137-1-ND
- C4: renamed from C1; Digikey Part Num (none) -> 1276-2928-1-ND
- C5: renamed from C2; Digikey Part Num (none) -> 1276-2928-1-ND
- C6: renamed from C4; footprint (none) -> Capacitor_THT:C_Radial_D6.3mm_H7.0mm_P2.50mm; Digikey Part Num (none) -> 1189-2182-ND
- C7: renamed from C?; footprint (none) -> Capacitor_SMD:C_0603_1608Metric; Digikey Part Num (none) -> n/a
- J1: renamed from J?; footprint (none) -> Connector_JST:JST_PH_B6B-PH-K_1x06_P2.00mm_Vertical; Digikey Part Num (none) -> 455-1708-ND
- J10, J11, J12, J13, J6, J7, J8, J9: renamed from J?; footprint (none) -> Connector_JST:JST_XH_B2B-XH-A_1x02_P2.50mm_Vertical
- J14: renamed from J?; footprint (none) -> Connector_JST:JST_XH_S4B-XH-A_1x04_P2.50mm_Horizontal
- J2: renamed from J?; footprint (none) -> Connector_PinHeader_2.54mm:PinHeader_1x08_P2.54mm_Vertical
- J3: renamed from J1; footprint (none) -> Connector_IDC:IDC-Header_2x10_P2.54mm_Vertical
- J4: renamed from J?; footprint (none) -> Connector_JST:JST_SH_SM04B-SRSS-TB_1x04-1MP_P1.00mm_Horizontal
- J5: renamed from J?; footprint (none) -> Connector_USB:USB_A_Molex_67643_Horizontal; Digikey Part Num (none) -> WM14667-ND
- JP1, JP2, JP3, JP4, JP5: renamed from JP?; footprint (none) -> Jumper:SolderJumper-3_P1.3mm_Open_RoundedPad1.0x1.5mm
- M1, M2, M3, M4, M5: renamed from M?; footprint (none) -> Connector_PinHeader_2.54mm:PinHeader_1x03_P2.54mm_Vertical
- Q1: renamed from Q?; footprint (none) -> Package_TO_SOT_SMD:SOT-23; Digikey Part Num (none) -> DMMT5401-FDICT-ND
- Q2, Q3, Q4, Q5, Q6, Q7, Q8, Q9: renamed from Q?; footprint (none) -> Package_TO_SOT_SMD:SOT-23; Digikey Part Num (none) -> TSM210N02CXRFGCT-ND
- R1, R16, R2, R3, R4, R5, R6, R7, R8, R9: renamed from R?; footprint (none) -> Resistor_SMD:R_0603_1608Metric; Digikey Part Num (none) -> n/a
- R10: renamed from R1; Digikey Part Num (none) -> n/a
- R11, R13: renamed from R?; Digikey Part Num (none) -> n/a
- R12: renamed from R2; Digikey Part Num (none) -> n/a
- R14: renamed from R?; footprint (none) -> Resistor_SMD:R_0603_1608Metric; Digikey Part Num (none) -> 311-47.0KHRCT-ND
- R15: renamed from R?; footprint (none) -> Resistor_SMD:R_0603_1608Metric; Digikey Part Num (none) -> RMCF0603FT200RCT-ND
- R17: renamed from R?; Digikey Part Num (none) -> 311-8.45KHRCT-ND
- R18: renamed from R?; Digikey Part Num (none) -> RMCF0603FT1K82CT-ND
- R19: renamed from R?; footprint (none) -> Resistor_SMD:R_0603_1608Metric; Digikey Part Num (none) -> 311-20.0KHRCT-ND
- U1, U2, U6, U7: renamed from U?; footprint (none) -> Connector_JST:JST_PH_B3B-PH-K_1x03_P2.00mm_Vertical; Digikey Part Num (none) -> 455-1705-ND
- U10: renamed from U?; footprint (none) -> Connector_Molex:Molex_SPOX_5268-04A_1x04_P2.50mm_Horizontal; Digikey Part Num (none) -> 23-0022057045-ND
- U11: renamed from U?; footprint (none) -> Package_SO:TSSOP-16_4.4x5mm_P0.65mm; Digikey Part Num (none) -> 568-1061-1-ND
- U3: renamed from U1; value AP1117-33 -> 3.3V LDO; Digikey Part Num (none) -> ZLDO1117G33DICT-ND
- U4: renamed from U?; footprint (none) -> ArmElectronics_Footprints:Pololu_3730; Digikey Part Num (none) -> 2183-3730-ND
- U5: renamed from U?; footprint (none) -> ASTRA_Footprints:Teensy4.1; Digikey Part Num (none) -> 1568-DEV-16771-ND
- U8, U9: renamed from U?; footprint (none) -> ASTRA_Footprints:Power_Supply_32nd_Brick; Digikey Part Num (none) -> 285-2720-ND
- renumbered JP1 to JP6
Other:
- moved on the sheet: C1, C2, C3, C4, C5, C6, C7, J1, J10, J11, J12, J13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

Commit message: Started PCB
Parts:
- removed BT1: Battery, Connector_AMASS:AMASS_XT60-M_1x02_P7.20mm_Vertical, symbol Device:Battery
- removed U4: Pololu_3730, ArmElectronics_Footprints:Pololu_3730, symbol ArmElectronics_Library:Pololu_3730
- added BT1: XT60_Battery_Connector, Connector_AMASS:AMASS_XT60-M_1x02_P7.20mm_Vertical, symbol ASTRA_Library:XT60_Battery_Connector
- added C8: 100uF, Capacitor_THT:C_Radial_D6.3mm_H7.0mm_P2.50mm, symbol Device:CP_Small
- added U4: Pololu_Compact_TB67S249FTG, ASTRA_Footprints:DIP-16_500, symbol ASTRA_Library:Pololu_Compact_TB67S249FTG
- J10, J11, J12, J13, J2, J4, J6, J7, J8, J9, JP1, JP2, JP3, JP4, JP5, JP6, M1, M2, M3, M4, M5: Digikey Part Num (none) -> n/a
- J14: footprint Connector_JST:JST_XH_S4B-XH-A_1x04_P2.50mm_Horizontal -> Connector_JST:JST_XH_B4B-XH-A_1x04_P2.50mm_Vertical; Digikey Part Num (none) -> n/a
- J3: Digikey Part Num (none) -> S9172-ND
- Q1: footprint Package_TO_SOT_SMD:SOT-23 -> Package_TO_SOT_SMD:SOT-23-6
- R16: value 10k -> 113k; Digikey Part Num n/a -> 311-113KHRCT-ND
- R19: value 20k -> 10k; Digikey Part Num 311-20.0KHRCT-ND -> n/a
Connections:
- net labels added: STEP_DMODE0, STEP_DMODE1, STEP_DMODE2, V_BAT_Div
- net labels removed: STEP_BEMF_DIV, STEP_CS, STEP_FAULT, STEP_STALL, STEP_~ENABLE~
- no-connect marks 10 -> 9
Other:
- moved on the sheet: J14

Commit message: DONE (please)
Parts:
- added H1, H2, H3: MountingHole, MountingHole:MountingHole_3.2mm_M3, symbol Mechanical:MountingHole
- J1: footprint Connector_JST:JST_PH_B6B-PH-K_1x06_P2.00mm_Vertical -> Connector_JST:JST_PH_S6B-PH-K_1x06_P2.00mm_Horizontal
Connections:
- net TEENSY_3.3 is gone; now on net +3V3: U5.28 (3.3V)
- net BULB: now also U5.46 (P39); no longer U5.26 (P22)
- net CLR_DATA: now also U5.38 (P31); no longer U5.35 (P28)
- net CLR_PIX: now also U5.35 (P28); no longer U5.37 (P30)
- net DATA_RDY: now also U5.37 (P30); no longer U5.32 (P25)
- net LED1: now also U5.48 (P41); no longer U5.41 (P34)
- net LED2: now also U5.47 (P40); no longer U5.42 (P35)
- net M1_PWM: now also U5.8 (P6); no longer U5.4 (P2)
- net M2_PWM: now also U5.7 (P5); no longer U5.5 (P3)
- net M4_PWM: now also U5.9 (P7); no longer U5.7 (P5)
- net M5_PWM: now also U5.10 (P8); no longer U5.8 (P6)
- net MOSFET1: now also U5.4 (P2); no longer U5.9 (P7)
- net MOSFET2: now also U5.5 (P3); no longer U5.10 (P8)
- net MOSFET3: now also U5.26 (P22); no longer U5.11 (P9)
- net MOSFET4: now also U5.19 (P15); no longer U5.39 (P32)
- net MOSFET5: now also U5.18 (P14); no longer U5.40 (P33)
- net PWR_DOWN: now also U5.39 (P32); no longer U5.31 (P24)
- net QWIIC_SCL: now also R12.2, U5.23 (P19); no longer R11.2, U5.20 (P16)
- net QWIIC_SDA: now also R10.2, U5.22 (P18); no longer R13.2, U5.21 (P17)
- net READ: now also U5.11 (P9); no longer U5.38 (P31)
- net SCL: now also R11.2, U5.20 (P16); no longer R12.2, U5.23 (P19)
- net SDA: now also R13.2, U5.21 (P17); no longer R10.2, U5.22 (P18)
- net STEP_DIR: now also U5.40 (P33); no longer U5.44 (P37)
- net STEP_DMODE0: now also U5.44 (P37); no longer U5.45 (P38)
- net STEP_DMODE1: now also U5.43 (P36); no longer U5.46 (P39)
- net STEP_DMODE2: now also U5.42 (P35); no longer U5.47 (P40)
- net STEP_STEP: now also U5.41 (P34); no longer U5.43 (P36)
- net VIDEO_N: now also U5.32 (P25); no longer U5.19 (P15)
- net VIDEO_P: now also U5.31 (P24); no longer U5.18 (P14)
- net V_BAT_Div: now also U5.45 (P38); no longer U5.48 (P41)
Changed lines of the file:
@@
 Wire Wire Line
 	10550 2900 10550 3050
-Wire Wire Line
-	2850 1550 2800 1550
 $Comp
 L power:+5V #PWR080
@@
 L power:GND #PWR089
 U 1 1 61203FD9
-P 3400 1700
-F 0 "#PWR089" H 3400 1450 50  0001 C CNN
-F 1 "GND" H 3400 1550 50  0000 C CNN
-F 2 "" H 3400 1700 50  0000 C CNN
-F 3 "" H 3400 1700 50  0000 C CNN
-	1    3400 1700
+P 3400 1450
+F 0 "#PWR089" H 3400 1200 50  0001 C CNN
+F 1 "GND" H 3400 1300 50  0000 C CNN
+F 2 "" H 3400 1450 50  0000 C CNN
+F 3 "" H 3400 1450 50  0000 C CNN
+	1    3400 1450
 	1    0    0    -1
 $EndComp
 Wire Wire Line
 	2800 1450 3400 1450
-Wire Wire Line
-	3400 1450 3400 1700
 Text Label 1900 2650 2    60   ~ 0
 ADC_DATA
 Text Label 2800 2650 0    60   ~ 0
 ADC_CLK
-Text Label 1900 2850 2    60   ~ 0
+Text Label 1900 3650 2    60   ~ 0
 PWR_DOWN
-Text Label 1900 2950 2    60   ~ 0
+Text Label 1900 3450 2    60   ~ 0
 DATA_RDY
-Text Label 1900 3250 2    60   ~ 0
+Text Label 1900 3550 2    60   ~ 0
 CLR_DATA
 Text Label 1900 3350 2    60   ~ 0
 SHUTTER
-Text Label 1900 3450 2    60   ~ 0
+Text Label 1900 3250 2    60   ~ 0
 CLR_PIX
-Text Label 1900 3550 2    60   ~ 0
+Text Label 1900 2350 2    60   ~ 0
 READ
 Text Label 1900 2450 2    60   ~ 0
 ADC_CS
-Text Label 2800 2550 0    60   ~ 0
+Text Label 1900 2850 2    60   ~ 0
 VIDEO_P
-Text Label 2800 2450 0    60   ~ 0
+Text Label 1900 2950 2    60   ~ 0
 VIDEO_N
-Text Label 2800 2050 0    60   ~ 0
+Text Label 2800 2350 0    60   ~ 0
 SCL
-Text Label 2800 2150 0    60   ~ 0
+Text Label 2800 2250 0    60   ~ 0
 SDA
 $Comp
@@
 Wire Wire Line
 	2800 2750 3550 2750
-Text Label 10050 6800 2    50   ~ 0
+Text Label 10300 7850 0    50   ~ 0
 SDA
-Text Label 10300 6800 0    50   ~ 0
+Text Label 10050 7850 2    50   ~ 0
 SCL
-Text Label 2850 1550 0    50   ~ 0
-TEENSY_3.3
 $Comp
 L Device:R_Small R12
@@
 Text Label 8000 10600 2    50   ~ 0
 QWIIC_SDA
-Text Label 2800 2350 0    50   ~ 0
+Text Label 2800 2050 0    50   ~ 0
 QWIIC_SCL
-Text Label 2800 2250 0    50   ~ 0
+Text Label 2800 2150 0    50   ~ 0
 QWIIC_SDA
 $Comp
@@
 F 0 "J1" H 6480 6542 50  0000 L CNN
 F 1 "Angle Sensor" H 6480 6451 50  0000 L CNN
-F 2 "Connector_JST:JST_PH_B6B-PH-K_1x06_P2.00mm_Vertical" H 6400 6550 50  0001 C CNN
+F 2 "Connector_JST:JST_PH_S6B-PH-K_1x06_P2.00mm_Horizontal" H 6400 6550 50  0001 C CNN
 F 3 "~" H 6400 6550 50  0001 C CNN
 F 4 "455-1708-ND" H 6400 6550 50  0001 C CNN "Digikey Part Num"
@@
 Text Label 1900 3050 2    50   ~ 0
 COPI1
-Text Label 1900 3650 2    50   ~ 0
+Text Label 2800 2450 0    50   ~ 0
 MOSFET4
-Text Label 2800 3650 0    50   ~ 0
+Text Label 2800 2550 0    50   ~ 0
 MOSFET5
-Text Label 1900 2150 2    50   ~ 0
+Text Label 1900 1650 2    50   ~ 0
 MOSFET1
-Text Label 1900 2250 2    50   ~ 0
+Text Label 1900 1750 2    50   ~ 0
 MOSFET2
-Text Label 1900 2350 2    50   ~ 0
+Text Label 2800 1750 0    50   ~ 0
 MOSFET3
 NoConn ~ 1900 2550
-Text Label 1900 1650 2    50   ~ 0
+Text Label 1900 2050 2    50   ~ 0
 M1_PWM
-Text Label 1900 1750 2    50   ~ 0
+Text Label 1900 1950 2    50   ~ 0
 M2_PWM
 Text Label 1900 1850 2    50   ~ 0
 M3_PWM
-Text Label 1900 1950 2    50   ~ 0
+Text Label 1900 2150 2    50   ~ 0
 M4_PWM
-Text Label 1900 2050 2    50   ~ 0
+Text Label 1900 2250 2    50   ~ 0
 M5_PWM
+Text Label 2800 2850 0    50   ~ 0
+LED1
+Text Label 2800 2950 0    50   ~ 0
+LED2
 Text Label 2800 3550 0    50   ~ 0
-LED1
-Text Label 2800 3450 0    50   ~ 0
-LED2
-Text Label 2800 3350 0    50   ~ 0
 STEP_STEP
-Text Label 2800 3250 0    50   ~ 0
+Text Label 2800 3650 0    50   ~ 0
 STEP_DIR
-Text Label 2800 1750 0    50   ~ 0
+Text Label 2800 3050 0    50   ~ 0
 BULB
 $Comp
@@
 $EndComp
 Connection ~ 10050 7350
-Text Label 10050 7850 2    50   ~ 0
+Text Label 10300 6800 0    50   ~ 0
 QWIIC_SCL
-Text Label 10300 7850 0    50   ~ 0
+Text Label 10050 6800 2    50   ~ 0
 QWIIC_SDA
 $Comp
@@
 Text Label 6000 1950 2    50   ~ 0
 STEP_DMODE2
-Text Label 2800 3150 0    50   ~ 0
+Text Label 2800 3250 0    50   ~ 0
 STEP_DMODE0
-Text Label 2800 3050 0    50   ~ 0
+Text Label 2800 3350 0    50   ~ 0
 STEP_DMODE1
-Text Label 2800 2950 0    50   ~ 0
+Text Label 2800 3450 0    50   ~ 0
 STEP_DMODE2
 Text Label 9000 1500 0    50   ~ 0
@@
 Wire Wire Line
 	9000 1600 9000 1500
-Text Label 2800 2850 0    50   ~ 0
+Text Label 2800 3150 0    50   ~ 0
 V_BAT_Div
 $Comp
@@
 	1    0    0    -1
 $EndComp
+$Comp
+L Mechanical:MountingHole H1
+U 1 1 619B14A8
+P 1050 10400
+F 0 "H1" H 1150 10446 50  0000 L CNN
+F 1 "MountingHole" H 1150 10355 50  0000 L CNN
+F 2 "MountingHole:MountingHole_3.2mm_M3" H 1050 10400 50  0001 C CNN
+F 3 "~" H 1050 10400 50  0001 C CNN
+	1    1050 10400
+	1    0    0    -1
+$EndComp
+$Comp
+L Mechanical:MountingHole H2
+U 1 1 619B4FAD
+P 1050 10600
+F 0 "H2" H 1150 10646 50  0000 L CNN
+F 1 "MountingHole" H 1150 10555 50  0000 L CNN
+F 2 "MountingHole:MountingHole_3.2mm_M3" H 1050 10600 50  0001 C CNN
+F 3 "~" H 1050 10600 50  0001 C CNN
+	1    1050 10600
+	1    0    0    -1
+$EndComp
+$Comp
+L Mechanical:MountingHole H3
+U 1 1 619B5149
+P 1050 10800
+F 0 "H3" H 1150 10846 50  0000 L CNN
+F 1 "MountingHole" H 1150 10755 50  0000 L CNN
+F 2 "MountingHole:MountingHole_3.2mm_M3" H 1050 10800 50  0001 C CNN
+F 3 "~" H 1050 10800 50  0001 C CNN
+	1    1050 10800
+	1    0    0    -1
+$EndComp
+$Comp
+L power:+3.3V #PWR0101
+U 1 1 61CEDF09
+P 3250 1550
+F 0 "#PWR0101" H 3250 1400 50  0001 C CNN
+F 1 "+3.3V" V 3250 1800 50  0000 C CNN
+F 2 "" H 3250 1550 50  0000 C CNN
+F 3 "" H 3250 1550 50  0000 C CNN
+	1    3250 1550
+	1    0    0    -1
+$EndComp
+Wire Wire Line
+	2800 1550 3250 1550
 $EndSCHEMATC

Commit message: started on V2
Parts:
- removed J10, J11, J12, J8, J9: Conn_01x02, Connector_JST:JST_XH_B2B-XH-A_1x02_P2.50mm_Vertical, symbol Connector_Generic:Conn_01x02
- removed JP3, JP4, JP5: SolderJumper_3_Open, Jumper:SolderJumper-3_P1.3mm_Open_RoundedPad1.0x1.5mm, symbol Jumper:SolderJumper_3_Open
- removed Q4, Q5, Q6, Q7, Q8: Q_NMOS_GSD, Package_TO_SOT_SMD:SOT-23, symbol Device:Q_NMOS_GSD
- removed R4, R5, R6, R7, R8: 10k, Resistor_SMD:R_0603_1608Metric, symbol Device:R_Small
- added J? (x2): Conn_01x02, Connector_JST:JST_XH_B2B-XH-A_1x02_P2.50mm_Vertical, symbol Connector_Generic:Conn_01x02
- added M6, M7, M8: Motor_Servo, Connector_PinHeader_2.54mm:PinHeader_1x03_P2.54mm_Vertical, symbol Motor:Motor_Servo
- added Q? (x2): Q_NMOS_GSD, Package_TO_SOT_SMD:SOT-23, symbol Device:Q_NMOS_GSD
- added R? (x2): 10k, Resistor_SMD:R_0603_1608Metric, symbol Device:R_Small
- added U? (x4): MAX14870_Breakout, symbol MainElectronicsLib:MAX14870_Breakout
- renumbered C2 to C1, C3 to C2, C8 to C3, C1 to C4, C4 to C5, C5 to C6, C6 to C8, J3 to J1, J13 to J14, J1 to J2, J2 to J3, J14 to J4, J4 to J5, J5 to J6, J6 to J7, J7 to J8, JP6 to JP1, JP1 to JP2, JP2 to JP3, Q9 to Q10, Q10 to Q2, Q2 to Q3, Q3 to Q4, R17 to R1, R15 to R10, R14 to R11, R2 to R12, R3 to R13, R9 to R19, R18 to R2, R16 to R3, R19 to R4, R10 to R5, R11 to R6, R1 to R7, R12 to R8, R13 to R9, U5 to U1, U6 to U10, U7 to U11, U4 to U2, U8 to U3, U9 to U4, U10 to U5, U11 to U6, U3 to U7, U1 to U8, U2 to U9
Connections:
- net +12V: now also J?.1 (Pin_1), J?.1 (Pin_1)
- net +5VP: now also M6.2 (+), M7.2 (+), M8.2 (+)
- net GND: now also M6.3 (-), M7.3 (-), M8.3 (-), Q?.2 (S), Q?.2 (S), R?.2, R?.2
- net M1_PWM: no longer U1.8 (P6)
- net M2_PWM: no longer U1.7 (P5)
- net M3_PWM: no longer U1.6 (P4)
- net M4_PWM: no longer U1.9 (P7)
- net M5_PWM: no longer U1.10 (P8)
- net BULB renamed FAN1
- net FAN1: no longer U1.46 (P39)
- net LED1: no longer names the net of U1.48 (P41)
- net LED2: no longer names the net of U1.47 (P40)
- net MOSFET1 renamed LIGHT1
- net LIGHT1: no longer U1.4 (P2)
- net MOSFET2 renamed LIGHT2
- net LIGHT2: no longer U1.5 (P3)
- net MOSFET3: no longer names the net of U1.26 (P22)
- net MOSFET4: no longer names the net of U1.19 (P15)
- net MOSFET5: no longer names the net of U1.18 (P14)
- new net: J?.2 (Pin_2), Q?.3 (D) (x2)
- new net FAN2: Q?.1 (G), R?.1
- new net FAN3: Q?.1 (G), R?.1
- new net M6_PWM: M6.1 (PWM)
- new net M7_PWM: M7.1 (PWM)
- new net M8_PWM: M8.1 (PWM)
Other:
- moved on the sheet: C3, J14, J4, J7, J8, JP2, JP3, M1, M2, M3, M4, M5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

Commit message: PCB Layout
Parts:
- removed C7: 0.1u, Capacitor_SMD:C_0603_1608Metric, symbol Device:C_Small
- removed J2: Angle Sensor, Connector_JST:JST_PH_S6B-PH-K_1x06_P2.00mm_Horizontal, symbol Connector_Generic:Conn_01x06
- removed J3: Conn_01x08, Connector_PinHeader_2.54mm:PinHeader_1x08_P2.54mm_Vertical, symbol Connector_Generic:Conn_01x08
- removed M7, M8: Motor_Servo, Connector_PinHeader_2.54mm:PinHeader_1x03_P2.54mm_Vertical, symbol Motor:Motor_Servo
- removed R3: 113k, Resistor_SMD:R_0603_1608Metric, symbol Device:R_Small
- removed R4: 10k, Resistor_SMD:R_0603_1608Metric, symbol Device:R_Small
- removed U11: AH1815-P-B, Connector_JST:JST_PH_B3B-PH-K_1x03_P2.00mm_Vertical, symbol ArmElectronics_Library:AH1815-P-B
- removed U6: PCA9557, Package_SO:TSSOP-16_4.4x5mm_P0.65mm, symbol ASTRA_Library:PCA9557
- removed U? (x3): MAX14870_Breakout, symbol MainElectronicsLib:MAX14870_Breakout
- added C3, C4: 0.1u, Capacitor_SMD:C_0603_1608Metric, symbol Device:C_Small
- added C5, C6: 22u, Capacitor_SMD:CP_Elec_6.3x5.9, symbol Device:CP_Small
- added H4: MountingHole, MountingHole:MountingHole_3.2mm_M3, symbol Mechanical:MountingHole
- added J10, J11, J12, J13, J14, J9: Conn_01x02, Connector_JST:JST_XH_B2B-XH-A_1x02_P2.50mm_Vertical, symbol Connector_Generic:Conn_01x02
- added JP3, JP5: SolderJumper_3_Open, Jumper:SolderJumper-3_P1.3mm_Open_RoundedPad1.0x1.5mm, symbol Jumper:SolderJumper_3_Open
- added Q8, Q9: Q_NMOS_GSD, Package_TO_SOT_SMD:SOT-23, symbol Device:Q_NMOS_GSD
- added R15, R16: 10k, Resistor_SMD:R_0603_1608Metric, symbol Device:R_Small
- added U10, U11, U9: MAX14870_Breakout, ASTRA_Footprints:Pololu_2961, symbol MainElectronicsLib:MAX14870_Breakout
- C1, C2: footprint Capacitor_SMD:CP_Elec_8x5.4 -> Capacitor_SMD:CP_Elec_10x10; Digikey Part Num 493-2137-1-ND -> 493-4402-1-ND
- J15: renamed from J4; Digikey Part Num n/a -> (none)
- J3: renamed from J5; Digikey Part Num n/a -> (none)
- J4: renamed from J14; Digikey Part Num n/a -> (none)
- J5, J6: renamed from J?; Digikey Part Num n/a -> (none)
- J7, J8, M1, M2, M3, M4, M5, M6: Digikey Part Num n/a -> (none)
- JP1: renamed from JP2; Digikey Part Num n/a -> (none)
- JP2: renamed from JP3; Digikey Part Num n/a -> (none)
- JP4: renamed from JP1; Digikey Part Num n/a -> (none)
- R1: renamed from R5; Digikey Part Num n/a -> (none)
- R10, R9: renamed from R?; Digikey Part Num n/a -> (none)
- R11: renamed from R7; Digikey Part Num n/a -> (none)
- R13: renamed from R12; Digikey Part Num n/a -> (none)
- R14: renamed from R13; Digikey Part Num n/a -> (none)
- R2: renamed from R6; Digikey Part Num n/a -> (none)
- R3: renamed from R8; Digikey Part Num n/a -> (none)
- R4: renamed from R9; Digikey Part Num n/a -> (none)
- R8: renamed from R19; Digikey Part Num n/a -> (none)
- U8: renamed from U?; footprint (none) -> ASTRA_Footprints:Pololu_2961; Digikey Part Num (none) -> 2183-2961-ND
- gave numbers to parts that had none: 2
- renumbered C8 to C10, C3 to C11, C4 to C7, C5 to C8, C6 to C9, J6 to J2, Q10 to Q1, Q1 to Q4, Q2 to Q5, Q3 to Q6, Q4 to Q7, R11 to R12, R10 to R5, R1 to R6, R2 to R7, U2 to U12, U10 to U13, U3 to U2, U4 to U3, U5 to U4, U7 to U5, U8 to U6, U9 to U7
Connections:
- net Angle_CS is gone; now on net Hall_SW_1: U1.27 (P23)
- net CIPO1 is gone; now on net M2_PWM: U1.3 (P1)
- net COPI1 is gone; now on net VIDEO_P: U1.33 (P26)
- net LIGHT1 is gone; now on net LIGHT: Q6.1 (G), R13.1
- net LIGHT2 is gone; now on net GEN1: Q7.1 (G), R14.1
- net SCK1 is gone; now on net VIDEO_N: U1.34 (P27)
- net +12V: now also U8.7 (VIN), C4.1, C6.1, JP3.1 (A), JP5.1 (A), U10.7 (VIN), U11.7 (VIN), U9.7 (VIN); no longer R7.1
- net +3V3: now also U12.2 (DMODE0), U12.3 (DMODE1), U12.4 (DMODE2)
- net +5VP: now also C3.1, C5.1, JP3.3 (B), JP5.3 (B); no longer R6.1
- net FAN1: now also U1.46 (P39)
- net FAN2: now also U1.44 (P37)
- net FAN3: now also U1.42 (P35)
- net GND: now also R6.2, R7.2, U8.5 (GND), U8.6 (GND), C3.2, C4.2, C5.2, C6.2, Q8.2 (S), Q9.2 (S), R15.2, R16.2, U10.5 (GND), U10.6 (GND), U11.5 (GND), U11.6 (GND), U9.5 (GND), U9.6 (GND)
- net Hall_SW_2: now also U1.26 (P22)
- net Hall_SW_3: now also U1.18 (P14)
- net M1_PWM: now also U1.2 (P0)
- net M3_PWM: now also U1.4 (P2)
- net M4_PWM: now also U1.5 (P3)
- net M5_PWM: now also U1.6 (P4)
- net M6_PWM: now also U1.7 (P5)
- net VIDEO_N: no longer U1.32 (P25)
- net VIDEO_P: no longer U1.31 (P24)
- net at U2.6 (TRIM): now also R6.1; no longer R6.2
- net at U3.6 (TRIM): now also R7.1; no longer R7.2
- net Pump2_PWM: now reaches U1.10 (P8)
- net Pump2_PWM: now also U10.1 (PWM)
- net Pump1_PWM: now reaches U1.19 (P15)
- net Pump1_PWM: now also U9.1 (PWM)
- net GEN1: now reaches U1.47 (P40)
- net LIGHT: now reaches U1.48 (P41)
- net Act_DIR: now reaches U1.8 (P6)
- net Act_DIR: now also U8.2 (DIR)
- net Act_PWM: now reaches U1.9 (P7)
- net Act_PWM: now also U8.1 (PWM)
- net at U8.8 (M2): now also J11.2 (Pin_2)
- net at U8.9 (M1): now also J11.1 (Pin_1)
- removed net STEP_DMODE0: U1.44 (P37), U12.2 (DMODE0)
- net STEP_DMODE1 renamed GEN3
- net GEN3: now also Q9.1 (G), R16.1; no longer U12.3 (DMODE1)
- removed net STEP_DMODE2: U1.42 (P35), U12.4 (DMODE2)
- net V_BAT_Div renamed GEN2
- net GEN2: now also Q8.1 (G), R15.1
- new net: J12.2 (Pin_2), U9.8 (M2)
- new net: J12.1 (Pin_1), U9.9 (M1)
- new net: J13.2 (Pin_2), U10.8 (M2)
- new net: J13.1 (Pin_1), U10.9 (M1)
- new net: J14.2 (Pin_2), U11.8 (M2)
- new net: J14.1 (Pin_1), U11.9 (M1)
- new net: J9.2 (Pin_2), Q8.3 (D)
- new net: J9.1 (Pin_1), JP3.2 (C)
- new net: J10.2 (Pin_2), Q9.3 (D)
- new net: J10.1 (Pin_1), JP5.2 (C)
- new net Pump3_PWM: U1.31 (P24), U11.1 (PWM)
- new net Pump_DIR: U1.32 (P25), U10.2 (DIR), U11.2 (DIR), U9.2 (DIR)
- no-connect marks 9 -> 21
Other:
- moved on the sheet: BT1, C1, C10, C11, C2, C7, C8, C9, J15, J2, J3, J4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
