File: adapter-shield/adapter-shield.kicad_pcb (KiCad board)
At the start: 2 copper layers, 7 parts, among them J1 Camera, U1 AP1117-33

Commit message: Started PCB
Parts:
- added BT1: XT60_Battery_Connector, Connector_AMASS:AMASS_XT60-M_1x02_P7.20mm_Vertical, F.Cu at (192.3, 106.0)
- added C5: 1uF, Capacitor_SMD:C_0805_2012Metric, F.Cu at (156.3, 107.7)
- added C6: 100uF, Capacitor_THT:C_Radial_D6.3mm_H7.0mm_P2.50mm, F.Cu at (204.7, 132.6)
- added C7: 0.1u, Capacitor_SMD:C_0603_1608Metric, F.Cu at (214.6, 124.1)
- added C8: 100uF, Capacitor_THT:C_Radial_D6.3mm_H7.0mm_P2.50mm, F.Cu at (180.8, 80.6)
- added J10: Conn_01x02, Connector_JST:JST_XH_B2B-XH-A_1x02_P2.50mm_Vertical, F.Cu at (233.0, 87.6)
- added J11: Conn_01x02, Connector_JST:JST_XH_B2B-XH-A_1x02_P2.50mm_Vertical, F.Cu at (233.0, 95.4)
- added J12: Conn_01x02, Connector_JST:JST_XH_B2B-XH-A_1x02_P2.50mm_Vertical, F.Cu at (191.8, 124.4)
- added J13: Conn_01x02, Connector_JST:JST_XH_B2B-XH-A_1x02_P2.50mm_Vertical, F.Cu at (196.0, 132.2)
- added J14: Conn_01x04, Connector_JST:JST_XH_B4B-XH-A_1x04_P2.50mm_Vertical, F.Cu at (213.8, 77.7)
- added J2: Conn_01x08, Connector_PinHeader_2.54mm:PinHeader_1x08_P2.54mm_Vertical, F.Cu at (166.3, 108.5)
- added J3: Camera, Connector_IDC:IDC-Header_2x10_P2.54mm_Vertical, F.Cu at (147.3, 80.5)
- added J4: QWIIC_Generic_Conn, Connector_JST:JST_SH_SM04B-SRSS-TB_1x04-1MP_P1.00mm_Horizontal, F.Cu at (215.0, 119.1)
- added J5: USB_A, Connector_USB:USB_A_Molex_67643_Horizontal, F.Cu at (174.3, 109.5)
- added J6: Conn_01x02, Connector_JST:JST_XH_B2B-XH-A_1x02_P2.50mm_Vertical, F.Cu at (219.3, 101.0)
- added J7: Conn_01x02, Connector_JST:JST_XH_B2B-XH-A_1x02_P2.50mm_Vertical, F.Cu at (214.0, 110.8)
- added J8: Conn_01x02, Connector_JST:JST_XH_B2B-XH-A_1x02_P2.50mm_Vertical, F.Cu at (202.2, 124.2)
- added J9: Conn_01x02, Connector_JST:JST_XH_B2B-XH-A_1x02_P2.50mm_Vertical, F.Cu at (186.6, 135.1)
- added JP2: SolderJumper_3_Open, Jumper:SolderJumper-3_P1.3mm_Open_RoundedPad1.0x1.5mm, F.Cu at (185.9, 141.3)
- added JP3: SolderJumper_3_Open, Jumper:SolderJumper-3_P1.3mm_Open_RoundedPad1.0x1.5mm, F.Cu at (241.8, 85.9)
- added JP4: SolderJumper_3_Open, Jumper:SolderJumper-3_P1.3mm_Open_RoundedPad1.0x1.5mm, F.Cu at (164.8, 140.3)
- added JP5: SolderJumper_3_Open, Jumper:SolderJumper-3_P1.3mm_Open_RoundedPad1.0x1.5mm, F.Cu at (170.4, 140.3)
- added JP6: Jumper, Connector_PinHeader_2.54mm:PinHeader_1x03_P2.54mm_Vertical, F.Cu at (227.2, 86.6)
- added M1: Motor_Servo, Connector_PinHeader_2.54mm:PinHeader_1x03_P2.54mm_Vertical, F.Cu at (180.8, 134.1)
- added M2: Motor_Servo, Connector_PinHeader_2.54mm:PinHeader_1x03_P2.54mm_Vertical, F.Cu at (208.2, 109.8)
- added M3: Motor_Servo, Connector_PinHeader_2.54mm:PinHeader_1x03_P2.54mm_Vertical, F.Cu at (201.1, 113.5)
- added M4: Motor_Servo, Connector_PinHeader_2.54mm:PinHeader_1x03_P2.54mm_Vertical, F.Cu at (222.6, 90.3)
- added M5: Motor_Servo, Connector_PinHeader_2.54mm:PinHeader_1x03_P2.54mm_Vertical, F.Cu at (239.0, 76.7)
- added Q1: Q_DUAL_PNP_PNP_C1B1B2C2E2E1, Package_TO_SOT_SMD:SOT-23-6, F.Cu at (243.5, 81.2)
- added Q10: Q_PMOS_GSD, Package_TO_SOT_SMD:SOT-23, F.Cu at (199.2, 138.9)
- added Q2: Q_NMOS_GSD, Package_TO_SOT_SMD:SOT-23, F.Cu at (175.5, 140.8)
- added Q3: Q_NMOS_GSD, Package_TO_SOT_SMD:SOT-23, F.Cu at (243.5, 76.7)
- added Q4: Q_NMOS_GSD, Package_TO_SOT_SMD:SOT-23, F.Cu at (241.2, 90.2)
- added Q5: Q_NMOS_GSD, Package_TO_SOT_SMD:SOT-23, F.Cu at (194.8, 138.9)
- added Q6: Q_NMOS_GSD, Package_TO_SOT_SMD:SOT-23, F.Cu at (210.4, 125.2)
- added Q7: Q_NMOS_GSD, Package_TO_SOT_SMD:SOT-23, F.Cu at (241.2, 94.8)
- added Q8: Q_NMOS_GSD, Package_TO_SOT_SMD:SOT-23, F.Cu at (222.2, 114.3)
- added Q9: Q_NMOS_GSD, Package_TO_SOT_SMD:SOT-23, F.Cu at (212.5, 96.8)
- added R1: 10k, Resistor_SMD:R_0603_1608Metric, F.Cu at (204.0, 137.8)
- added R10: 10k, Resistor_SMD:R_0603_1608Metric, F.Cu at (226.9, 95.2)
- added R11: 10k, Resistor_SMD:R_0603_1608Metric, F.Cu at (190.3, 130.1)
- added R12: 10k, Resistor_SMD:R_0603_1608Metric, F.Cu at (216.8, 95.8)
- added R13: 10k, Resistor_SMD:R_0603_1608Metric, F.Cu at (176.3, 127.3)
- added R14: 47k, Resistor_SMD:R_0603_1608Metric, F.Cu at (176.3, 124.8)
- added R15: 200, Resistor_SMD:R_0603_1608Metric, F.Cu at (211.9, 129.2)
- added R16: 113k, Resistor_SMD:R_0603_1608Metric, F.Cu at (180.2, 85.8)
- added R17: 8.45k, Resistor_SMD:R_0603_1608Metric, F.Cu at (226.5, 113.3)
- added R18: 1.82k, Resistor_SMD:R_0603_1608Metric, F.Cu at (198.8, 142.4)
- added R19: 10k, Resistor_SMD:R_0603_1608Metric, F.Cu at (180.2, 88.3)
- added R2: 10k, Resistor_SMD:R_0603_1608Metric, F.Cu at (238.6, 101.1)
- added R3: 10k, Resistor_SMD:R_0603_1608Metric, F.Cu at (230.8, 111.5)
- added R4: 10k, Resistor_SMD:R_0603_1608Metric, F.Cu at (241.0, 98.3)
- added R5: 10k, Resistor_SMD:R_0603_1608Metric, F.Cu at (230.8, 109.0)
- added R6: 10k, Resistor_SMD:R_0603_1608Metric, F.Cu at (194.8, 142.4)
- added R7: 10k, Resistor_SMD:R_0603_1608Metric, F.Cu at (190.8, 142.4)
- added R8: 10k, Resistor_SMD:R_0603_1608Metric, F.Cu at (205.4, 118.4)
- added R9: 10k, Resistor_SMD:R_0603_1608Metric, F.Cu at (179.7, 142.7)
- added U10: LynxServo, Connector_Molex:Molex_SPOX_5268-04A_1x04_P2.50mm_Horizontal, F.Cu at (167.5, 130.9)
- added U11: PCA9557, Package_SO:TSSOP-16_4.4x5mm_P0.65mm, F.Cu at (224.4, 108.7)
- added U2: AH1815-P-B, Connector_JST:JST_PH_B3B-PH-K_1x03_P2.00mm_Vertical, F.Cu at (145.0, 138.8)
- added U3: 3.3V LDO, Package_TO_SOT_SMD:SOT-223-3_TabPin2, F.Cu at (183.4, 127.6)
- added U4: Pololu_Compact_TB67S249FTG, ASTRA_Footprints:DIP-16_500, F.Cu at (167.4, 85.0)
- added U5: Teensy_4.1, ASTRA_Footprints:Teensy4.1, F.Cu at (123.7, 135.9)
- added U6: AH1815-P-B, Connector_JST:JST_PH_B3B-PH-K_1x03_P2.00mm_Vertical, F.Cu at (213.3, 90.7)
- added U7: AH1815-P-B, Connector_JST:JST_PH_B3B-PH-K_1x03_P2.00mm_Vertical, F.Cu at (208.9, 103.6)
- added U8: TDK_I3A4W008A033V, ASTRA_Footprints:Power_Supply_32nd_Brick, F.Cu at (146.2, 115.2)
- added U9: TDK_I3A4W008A033V, ASTRA_Footprints:Power_Supply_32nd_Brick, F.Cu at (192.5, 80.0)
- C1: value 1uF -> 100uF; footprint Capacitor_SMD:C_0805_2012Metric -> Capacitor_THT:C_Radial_D6.3mm_H7.0mm_P2.50mm
- C2: value 1uF -> 33u; footprint Capacitor_SMD:C_0805_2012Metric -> Capacitor_SMD:CP_Elec_8x5.4
- C3: value 100uF -> 33u; footprint Capacitor_THT:CP_Radial_D5.0mm_P2.50mm -> Capacitor_SMD:CP_Elec_8x5.4
- C4: value 100uF -> 1uF; footprint Capacitor_THT:CP_Radial_D5.0mm_P2.50mm -> Capacitor_SMD:C_0805_2012Metric
- J1: value Camera -> Angle Sensor; footprint Connector_PinSocket_2.54mm:PinSocket_2x10_P2.54mm_Vertical -> Connector_JST:JST_PH_B6B-PH-K_1x06_P2.00mm_Vertical
- JP1: value Jumper -> SolderJumper_3_Open; footprint Connector_PinHeader_2.54mm:PinHeader_1x03_P2.54mm_Vertical -> Jumper:SolderJumper-3_P1.3mm_Open_RoundedPad1.0x1.5mm
- U1: value AP1117-33 -> AH1815-P-B; footprint Package_TO_SOT_SMD:SOT-223-3_TabPin2 -> Connector_JST:JST_PH_B3B-PH-K_1x03_P2.00mm_Vertical
- moved C3 88.7 mm to (230.8, 79.3)
- moved C1 85.2 mm to (231.4, 103.8), turned to 0 degrees
- moved J1 56.4 mm to (125.9, 139.4), turned to 0 degrees
- moved C2 52.6 mm to (192.9, 116.1), turned to 0 degrees
- moved JP1 40.0 mm to (171.5, 125.3), turned to 0 degrees
- moved U1 27.7 mm to (155.0, 138.8), turned to 0 degrees
- moved C4 16.0 mm to (160.7, 107.7)
Connections:
- C2 pad 1: Net-(C2-Pad1) -> /V_BAT
- C3 pad 1: +5V -> /V_BAT
- C4 pad 1: Net-(C2-Pad1) -> +5V
- J1 pad 1: GND -> +3V3
- J1 pad 2: (no net) -> GND
- J1 pad 3: (no net) -> /COPI1
- J1 pad 4: (no net) -> /CIPO1
- J1 pad 5: (no net) -> /SCK1
- J1 pad 6: (no net) -> /Angle_CS
- JP1 pad 1: (no net) -> +12V
- JP1 pad 2: +3V3 -> Net-(J6-Pad1)
- JP1 pad 3: Net-(C2-Pad1) -> +5VP
- U1 pad 1: GND -> +3V3
- U1 pad 2: Net-(C2-Pad1) -> GND
- U1 pad 3: +5V -> /Hall_SW_1
Routing:
- net Net-(C2-Pad1): track 19.0 -> 0.00 mm
- net GND: track 10.3 -> 0.00 mm, vias 9 -> 0
- net +3V3: track 8.07 -> 0.00 mm
- net +5V: track 6.52 -> 0.00 mm
- net (no net): track 1.11 -> 0.00 mm
- removed copper zone on F.Cu, net +3V3
- removed copper zone on B.Cu, net GND
Other:
- board text removed: "*GND"
- board text removed: "1"
- board text removed: "3.3V VCC"
- board text removed: "AVDD"
- board text removed: "AVSS"
- board text removed: "EPC901 Breakout to Shield Adapter"
- board text removed: "FRONT"
- board text removed: "HOST"
- board text removed: "LDO"
- board text removed: "Rev A"

Commit message: DONE (please)
Parts:
- added H1: MountingHole, MountingHole:MountingHole_3.2mm_M3, F.Cu at (113.0, 110.4)
- added H2: MountingHole, MountingHole:MountingHole_3.2mm_M3, F.Cu at (203.0, 110.4)
- added H3: MountingHole, MountingHole:MountingHole_3.2mm_M3, F.Cu at (203.0, 174.4)
- J1: footprint Connector_JST:JST_PH_B6B-PH-K_1x06_P2.00mm_Vertical -> Connector_JST:JST_PH_S6B-PH-K_1x06_P2.00mm_Horizontal
- JP1, JP2, JP3, JP4, JP5: moved to B.Cu
- moved JP6 121.8 mm to (118.0, 140.4), turned to 270 degrees
- moved Q1 118.7 mm to (132.5, 123.4)
- moved C1 117.2 mm to (115.0, 117.4), turned to 180 degrees
- moved J14 114.1 mm to (154.0, 174.9), turned to 180 degrees
- moved M5 101.4 mm to (152.5, 129.6), turned to 270 degrees
- moved R10 101.0 mm to (135.4, 138.0)
- moved J3 95.9 mm to (116.6, 171.4), turned to 180 degrees
- moved C6 91.7 mm to (113.0, 134.9)
- moved J4 91.4 mm to (124.0, 110.4), turned to 180 degrees
- moved R12 90.5 mm to (135.4, 135.4)
- moved Q3 89.4 mm to (162.0, 113.4)
- moved R19 88.7 mm to (135.3, 164.9), turned to 270 degrees
- moved R16 87.9 mm to (135.3, 161.4), turned to 270 degrees
- moved Q4 83.8 mm to (162.0, 117.4)
- moved R4 83.7 mm to (159.5, 117.4), turned to 270 degrees
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Connections:
- R10 pad 2: /SDA -> /QWIIC_SDA
- R11 pad 2: /QWIIC_SCL -> /SCL
- R12 pad 2: /SCL -> /QWIIC_SCL
- R13 pad 2: /QWIIC_SDA -> /SDA
- U5 pad 10: /MOSFET2 -> /M5_PWM
- U5 pad 11: /MOSFET3 -> /READ
- U5 pad 17: /VIDEO_P -> /ADC_CLK
- U5 pad 18: /ADC_CLK -> /MOSFET5
- U5 pad 19: /VIDEO_N -> /MOSFET4
- U5 pad 20: /QWIIC_SCL -> /SCL
- U5 pad 21: /QWIIC_SDA -> /SDA
- U5 pad 22: /SDA -> /QWIIC_SDA
- U5 pad 23: /SCL -> /QWIIC_SCL
- U5 pad 26: /BULB -> /MOSFET3
- U5 pad 28: /TEENSY_3.3 -> +3V3
- U5 pad 31: /PWR_DOWN -> /VIDEO_P
- U5 pad 32: /DATA_RDY -> /VIDEO_N
- U5 pad 35: /CLR_DATA -> /CLR_PIX
- U5 pad 37: /CLR_PIX -> /DATA_RDY
- U5 pad 38: /READ -> /CLR_DATA
- U5 pad 39: /MOSFET4 -> /PWR_DOWN
- U5 pad 4: /M1_PWM -> /MOSFET1
- U5 pad 40: /MOSFET5 -> /STEP_DIR
- U5 pad 41: /LED1 -> /STEP_STEP
- U5 pad 42: /LED2 -> /STEP_DMODE2
- U5 pad 43: /STEP_STEP -> /STEP_DMODE1
- U5 pad 44: /STEP_DIR -> /STEP_DMODE0
- U5 pad 45: /STEP_DMODE0 -> /V_BAT_Div
- U5 pad 46: /STEP_DMODE1 -> /BULB
- U5 pad 47: /STEP_DMODE2 -> /LED2
- U5 pad 48: /V_BAT_Div -> /LED1
- U5 pad 5: /M2_PWM -> /MOSFET2
- U5 pad 7: /M4_PWM -> /M2_PWM
- U5 pad 8: /M5_PWM -> /M1_PWM
- U5 pad 9: /MOSFET1 -> /M4_PWM
Routing:
- net +5VP: track 0.00 -> 248.9 mm, vias 0 -> 3
- net +3V3: track 0.00 -> 181.9 mm, vias 0 -> 4
- net +12V: track 0.00 -> 165.1 mm, vias 0 -> 2
- net /V_BAT: track 0.00 -> 69.9 mm
- net /SCK1: track 0.00 -> 58.8 mm, vias 0 -> 6
- net /COPI1: track 0.00 -> 58.4 mm, vias 0 -> 6
- net /BULB: track 0.00 -> 56.6 mm, vias 0 -> 2
- net /MOSFET2: track 0.00 -> 53.5 mm, vias 0 -> 3
- net /QWIIC_SCL: track 0.00 -> 53.1 mm, vias 0 -> 2
- net /QWIIC_SDA: track 0.00 -> 52.3 mm
- net /LED2: track 0.00 -> 50.5 mm, vias 0 -> 2
- net /MOSFET1: track 0.00 -> 50.4 mm, vias 0 -> 3
- net /LED1: track 0.00 -> 44.3 mm, vias 0 -> 2
- net +5V: track 0.00 -> 42.1 mm, vias 0 -> 2
- net /M1_PWM: track 0.00 -> 41.5 mm, vias 0 -> 3
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- added copper zone on F.Cu, net /V_BAT
- added copper zone on B.Cu, net GND
- added copper zone on F.Cu, net GND
Other:
- board outline added: 98 x 72 mm
- rule pad_to_mask_clearance: 0 -> 0.0508
- rule trace_min: 0.2 -> 0.1524
- rule via_min_drill: 0.3 -> 0.254
- rule via_min_size: 0.4 -> 0.508
- board text added: "1"
- board text added: "1 2 3 4 GND 12v 5v 3v3"
- board text added: "12V"
- board text added: "2"
- board text added: "3"
- board text added: "3 2 1 4 5"
- board text added: "4"
- board text added: "5"
- board text added: "5V"
- board text added: "Bulb"
- board text added: "EPC 3.3V"
- board text added: "LDO Teensy"
- board text added: "LED1"
- board text added: "LED2"
- board text added: "Servos"

Commit message: Added info
Other:
- board text added: "ASTRA Biosensor V1.5 Designed by Thomas Bennett 21 Sep 2021 Forked from Adrian Studer's EPC901 Adapter"

Commit message: PCB Layout
Parts:
- removed the C7 at (147.0, 139.4)
- removed the C8 at (162.0, 151.4)
- removed the J1 at (141.6, 113.2)
- removed the JP4 at (197.0, 112.4)
- removed the Q4 at (162.0, 117.4)
- removed the Q5 at (162.0, 121.4)
- removed R17: 8.45k, Resistor_SMD:R_0603_1608Metric
- removed R18: 1.82k, Resistor_SMD:R_0603_1608Metric
- removed R19: 10k, Resistor_SMD:R_0603_1608Metric
- removed the R2 at (159.5, 109.4)
- removed the R3 at (159.5, 113.4)
- removed the R4 at (159.5, 117.4)
- removed the U1 at (170.0, 145.9)
- added C1: 33u, Capacitor_SMD:CP_Elec_10x10, F.Cu at (227.0, 178.4)
- added C11: 100uF, Capacitor_THT:C_Radial_D6.3mm_H7.0mm_P2.50mm, F.Cu at (161.0, 179.4)
- added C4: 0.1u, Capacitor_SMD:C_0603_1608Metric, F.Cu at (214.0, 135.4)
- added C5: 22u, Capacitor_SMD:CP_Elec_6.3x5.9, F.Cu at (215.0, 178.4)
- added C6: 22u, Capacitor_SMD:CP_Elec_6.3x5.9, F.Cu at (213.0, 140.4)
- added H4: MountingHole, MountingHole:MountingHole_3.2mm_M3, F.Cu at (237.0, 181.4)
- added J15: Conn_01x04, Connector_JST:JST_XH_B4B-XH-A_1x04_P2.50mm_Vertical, F.Cu at (145.0, 179.4)
- added J4: Conn_01x02, Connector_JST:JST_XH_B2B-XH-A_1x02_P2.50mm_Vertical, F.Cu at (183.0, 169.4)
- added M6: Motor_Servo, Connector_PinHeader_2.54mm:PinHeader_1x03_P2.54mm_Vertical, F.Cu at (157.0, 139.4)
- added Q1: Q_NMOS_GSD, Package_TO_SOT_SMD:SOT-23, F.Cu at (184.0, 162.4)
- added R10: 10k, Resistor_SMD:R_0603_1608Metric, F.Cu at (167.4, 162.4)
- added R13: 10k, Resistor_SMD:R_0603_1608Metric, F.Cu at (188.4, 162.4)
- added R14: 10k, Resistor_SMD:R_0603_1608Metric, F.Cu at (182.9, 156.4)
- added U12: Pololu_Compact_TB67S249FTG, ASTRA_Footprints:DIP-16_500, F.Cu at (152.0, 166.9)
- added U13: AH1815-P-B, Connector_JST:JST_PH_B3B-PH-K_1x03_P2.00mm_Vertical, F.Cu at (145.0, 121.4)
- added U3: TDK_I3A4W008A033V, ASTRA_Footprints:Power_Supply_32nd_Brick, F.Cu at (227.0, 129.4)
- C2: footprint Capacitor_SMD:CP_Elec_8x5.4 -> Capacitor_SMD:CP_Elec_10x10
- C3: value 33u -> 0.1u; footprint Capacitor_SMD:CP_Elec_8x5.4 -> Capacitor_SMD:C_0603_1608Metric
- J14: value Conn_01x04 -> Conn_01x02; footprint Connector_JST:JST_XH_B4B-XH-A_1x04_P2.50mm_Vertical -> Connector_JST:JST_XH_B2B-XH-A_1x02_P2.50mm_Vertical
- J2: value Conn_01x08 -> USB_A; footprint Connector_PinHeader_2.54mm:PinHeader_1x08_P2.54mm_Vertical -> Connector_USB:USB_A_Molex_67643_Horizontal
- J5: value USB_A -> Conn_01x02; footprint Connector_USB:USB_A_Molex_67643_Horizontal -> Connector_JST:JST_XH_B2B-XH-A_1x02_P2.50mm_Vertical
- R15: value 200 -> 10k
- R16: value 113k -> 10k
- R5: value 10k -> 200
- R6: value 10k -> 8.45k
- R7: value 10k -> 1.82k
- U10: value LynxServo -> MAX14870_Breakout; footprint Connector_Molex:Molex_SPOX_5268-04A_1x04_P2.50mm_Horizontal -> ASTRA_Footprints:Pololu_2961
- U11: value PCA9557 -> MAX14870_Breakout; footprint Package_SO:TSSOP-16_4.4x5mm_P0.65mm -> ASTRA_Footprints:Pololu_2961
- U2: value AH1815-P-B -> TDK_I3A4W008A033V; footprint Connector_JST:JST_PH_B3B-PH-K_1x03_P2.00mm_Vertical -> ASTRA_Footprints:Power_Supply_32nd_Brick
- U4: value Pololu_Compact_TB67S249FTG -> LynxServo; footprint ASTRA_Footprints:DIP-16_500 -> Connector_Molex:Molex_SPOX_5268-04A_1x04_P2.50mm_Horizontal
- U8, U9: value TDK_I3A4W008A033V -> MAX14870_Breakout; footprint ASTRA_Footprints:Power_Supply_32nd_Brick -> ASTRA_Footprints:Pololu_2961
- moved H3 90.3 mm to (113.0, 181.4)
- moved J14 78.2 mm to (201.0, 112.4)
- moved U2 72.7 mm to (230.0, 167.4)
- moved JP1 69.0 mm to (193.0, 178.4), turned to 270 degrees
- moved J9 68.4 mm to (176.0, 178.4), turned to 270 degrees
- moved J7 67.1 mm to (190.0, 178.4), turned to 270 degrees
- moved JP3 66.8 mm to (179.0, 178.4), turned to 270 degrees
- moved JP2 66.2 mm to (186.0, 178.4), turned to 270 degrees
- moved J8 66.1 mm to (183.0, 178.4), turned to 270 degrees
- moved R5 62.5 mm to (202.6, 166.6), turned to 180 degrees
- moved J10 57.0 mm to (169.0, 178.4), turned to 270 degrees
- moved J6 57.0 mm to (169.0, 169.4), turned to 270 degrees
- moved JP5 57.0 mm to (172.0, 178.4), turned to 270 degrees
- moved R6 56.6 mm to (211.0, 155.4), turned to 90 degrees
- moved Q2 55.1 mm to (177.0, 162.4)
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- renumbered C6 to C10, C1 to C7, C4 to C8, C5 to C9, J3 to J1, J4 to J3, JP6 to JP4, Q1 to Q4, Q10 to Q5, R10 to R1, R1 to R11, R14 to R12, R11 to R2, R12 to R3, R13 to R4, U5 to U1, U3 to U5
Connections:
- C3 pad 1: /V_BAT -> +5VP
- J1 pad 10: /VDD_OA -> (no net)
- J1 pad 7: /GND_OA -> (no net)
- J11 pad 1: +12V -> Net-(J11-Pad1)
- J12 pad 1: +12V -> Net-(J12-Pad1)
- J13 pad 1: +12V -> Net-(J13-Pad1)
- J2 pad 1: +3V3 -> +5VP
- J2 pad 2: +5VP -> Net-(J2-Pad2)
- J2 pad 3: +12V -> Net-(J2-Pad3)
- J2 pad 5: /IO1 -> Net-(J2-Pad5)
- J5 pad 1: +5VP -> +12V
- J6 pad 1: Net-(J6-Pad1) -> +12V
- JP1 pad 2: Net-(J6-Pad1) -> Net-(J7-Pad1)
- JP2 pad 2: Net-(J7-Pad1) -> Net-(J8-Pad1)
- JP3 pad 2: Net-(J8-Pad1) -> Net-(J9-Pad1)
- Q2 pad 1: /MOSFET1 -> /FAN2
- Q2 pad 3: Net-(J6-Pad2) -> Net-(J5-Pad2)
- Q3 pad 1: /MOSFET2 -> /FAN3
- Q3 pad 3: Net-(J7-Pad2) -> Net-(J6-Pad2)
- Q6 pad 1: /MOSFET5 -> /LIGHT
- Q6 pad 3: Net-(J10-Pad2) -> Net-(J7-Pad2)
- Q7 pad 1: /LED1 -> /GEN1
- Q7 pad 3: Net-(J11-Pad2) -> Net-(J8-Pad2)
- Q8 pad 1: /LED2 -> /GEN2
- Q8 pad 3: Net-(J12-Pad2) -> Net-(J9-Pad2)
- Q9 pad 1: /BULB -> /GEN3
- Q9 pad 3: Net-(J13-Pad2) -> Net-(J10-Pad2)
- R15 pad 1: Net-(J5-Pad3) -> /GEN2
- R15 pad 2: Net-(J5-Pad2) -> GND
- R16 pad 1: /V_BAT -> /GEN3
- R16 pad 2: /V_BAT_Div -> GND
- R5 pad 1: /MOSFET4 -> Net-(J2-Pad3)
- R5 pad 2: GND -> Net-(J2-Pad2)
- R6 pad 1: /MOSFET5 -> Net-(R6-Pad1)
- R7 pad 1: /LED1 -> Net-(R7-Pad1)
- R8 pad 1: /LED2 -> /FAN1
- R9 pad 1: /BULB -> /FAN2
- U1 pad 10: /M5_PWM -> /Pump2_PWM
- U1 pad 13: Net-(U5-Pad13) -> (no net)
- U1 pad 18: /MOSFET5 -> /Hall_SW_3
- U1 pad 19: /MOSFET4 -> /Pump1_PWM
- U1 pad 2: Net-(U5-Pad2) -> /M1_PWM
- U1 pad 26: /MOSFET3 -> /Hall_SW_2
- U1 pad 27: /Angle_CS -> /Hall_SW_1
- U1 pad 3: /CIPO1 -> /M2_PWM
- U1 pad 31: /VIDEO_P -> /Pump3_PWM
- U1 pad 32: /VIDEO_N -> /Pump_DIR
- U1 pad 33: /COPI1 -> /VIDEO_P
- U1 pad 34: /SCK1 -> /VIDEO_N
- U1 pad 4: /MOSFET1 -> /M3_PWM
- U1 pad 42: /STEP_DMODE2 -> /FAN3
- U1 pad 43: /STEP_DMODE1 -> /GEN3
- U1 pad 44: /STEP_DMODE0 -> /FAN2
- U1 pad 45: /V_BAT_Div -> /GEN2
- U1 pad 46: /BULB -> /FAN1
- U1 pad 47: /LED2 -> /GEN1
- U1 pad 48: /LED1 -> /LIGHT
- U1 pad 5: /MOSFET2 -> /M4_PWM
- U1 pad 6: /M3_PWM -> /M5_PWM
- U1 pad 7: /M2_PWM -> /M6_PWM
- U1 pad 8: /M1_PWM -> /Act_DIR
- U1 pad 9: /M4_PWM -> /Act_PWM
- U10 pad 1: /Lynx_RX -> /Pump2_PWM
- U10 pad 2: +12V -> /Pump_DIR
- U10 pad 3: GND -> (no net)
- U10 pad 4: /Lynx_TX -> (no net)
- U11 pad 1: /QWIIC_SCL -> /Pump3_PWM
- U11 pad 10: /Hall_SW_4 -> (no net)
- U11 pad 2: /QWIIC_SDA -> /Pump_DIR
- U11 pad 3: GND -> (no net)
- U11 pad 4: GND -> (no net)
- U11 pad 6: /Hall_SW_1 -> GND
- U11 pad 7: /Hall_SW_2 -> +12V
- U11 pad 8: GND -> Net-(J14-Pad2)
- U11 pad 9: /Hall_SW_3 -> Net-(J14-Pad1)
- U2 pad 1: +3V3 -> /V_BAT
- U2 pad 2: GND -> (no net)
- U2 pad 3: /Hall_SW_2 -> GND
- U4 pad 1: Net-(U4-Pad1) -> /Lynx_RX
- U4 pad 2: /STEP_DMODE0 -> +12V
- U4 pad 3: /STEP_DMODE1 -> GND
- U4 pad 4: /STEP_DMODE2 -> /Lynx_TX
- U6 pad 3: /Hall_SW_3 -> /Hall_SW_1
- U7 pad 3: /Hall_SW_4 -> /Hall_SW_2
- U8 pad 1: /V_BAT -> /Act_PWM
- U8 pad 2: Net-(U8-Pad2) -> /Act_DIR
- U8 pad 3: GND -> (no net)
- U8 pad 4: GND -> (no net)
- U8 pad 5: Net-(U8-Pad5) -> GND
- U8 pad 6: Net-(R17-Pad2) -> GND
- U8 pad 7: +5VP -> +12V
- U8 pad 8: +5VP -> Net-(J11-Pad2)
- U9 pad 1: /V_BAT -> /Pump1_PWM
- U9 pad 2: Net-(U9-Pad2) -> /Pump_DIR
- U9 pad 3: GND -> (no net)
- U9 pad 4: GND -> (no net)
- U9 pad 5: Net-(U9-Pad5) -> GND
- U9 pad 6: Net-(R18-Pad2) -> GND
- U9 pad 8: +12V -> Net-(J12-Pad2)
Routing:
- net /Pump_DIR: track 0.00 -> 115.6 mm, vias 0 -> 3
- net /Pump2_PWM: track 0.00 -> 104.4 mm, vias 0 -> 2
- net /Act_DIR: track 0.00 -> 87.0 mm, vias 0 -> 2
- net /Pump3_PWM: track 0.00 -> 86.9 mm, vias 0 -> 2
- net /Act_PWM: track 0.00 -> 84.8 mm, vias 0 -> 2
- net +5VP: track 248.9 -> 168.8 mm, vias 3 -> 6
- net /M6_PWM: track 0.00 -> 71.8 mm
- net /LIGHT: track 0.00 -> 61.6 mm
- net /SCK1: track 58.8 -> 0.00 mm, vias 6 -> 0
- net /COPI1: track 58.4 -> 0.00 mm, vias 6 -> 0
- net /BULB: track 56.6 -> 0.00 mm, vias 2 -> 0
- net /FAN1: track 0.00 -> 56.6 mm
- net /MOSFET2: track 53.5 -> 0.00 mm, vias 3 -> 0
- net /Pump1_PWM: track 0.00 -> 52.2 mm, vias 0 -> 1
- net /FAN2: track 0.00 -> 52.1 mm
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- added copper zone on F.Cu, net +12V
- added copper zone on F.Cu, net +5VP
Other:
- board size 98 x 72 mm -> 132 x 79 mm
- board text removed: "1"
- board text removed: "1 2 3 4 GND 12v 5v 3v3"
- board text removed: "12V"
- board text removed: "2"
- board text removed: "3"
- board text removed: "3 2 1 4 5"
- board text removed: "4"
- board text removed: "5"
- board text removed: "5V"
- board text removed: "ASTRA Biosensor V1.5 Designed by Thomas Bennett 21 Sep 2021 Forked from Adrian Studer's EPC901 Adapter"
- board text removed: "Bulb"
- board text removed: "LED1"
- board text removed: "LED2"
- board text removed: "Servos"

Commit message: Finished PCB
Other:
- board text added: "1"
- board text added: "12V"
- board text added: "2"
- board text added: "3"
- board text added: "4"
- board text added: "5"
- board text added: "5V"
- board text added: "6"
- board text added: "ACTR"
- board text added: "FANS"
- board text added: "LIGHT"
- board text added: "Lim SW"
- board text added: "MAX14870 DRIVER"
- board text added: "MISC1"
- board text added: "MISC2"
- board text added: "MISC3"
- board text added: "PMP1"
- board text added: "PMP2"
- board text added: "PMP3"
- board text added: "S Vcc Gnd"
- board text added: "SERVOS"
- board text added: "SMART"
- board text added: "UAH SHC ASTRA Biosensor PCB V2 April 2022"
